File: Hardware/Board.sch (EAGLE design)
At the start: 55 parts, among them U1 EDISON_CONNECTOR_FULLMOUNTING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, U2 LAN9512-JZX, U4 EDISON_CONNECTOR_FULLHEADER, X1 J1011F01P

Commit message: Rolled back previous change
Parts:
- LED1: device led:LEDCHIPLED_0603 -> led:LEDCHIP-LED0805
Changed lines of the file:
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@@
 <part name="R11" library="resistor" deviceset="R-US_" device="R0402" value="330"/>
 <part name="R12" library="resistor" deviceset="R-US_" device="R0402" value="330"/>
-<part name="LED1" library="led" deviceset="LED" device="CHIPLED_0603" value="Green LED"/>
+<part name="LED1" library="led" deviceset="LED" device="CHIP-LED0805" value="Green LED"/>
 <part name="R13" library="resistor" deviceset="R-US_" device="R0402" value="330"/>
 <part name="+3V9" library="supply1" deviceset="+3V3" device=""/>

Commit message: Changed LED from 0805 package to 0603 package
Parts:
- LED1: device led:LEDCHIP-LED0805 -> led:LEDCHIPLED_0603
Changed lines of the file:
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@@
 <part name="R11" library="resistor" deviceset="R-US_" device="R0402" value="330"/>
 <part name="R12" library="resistor" deviceset="R-US_" device="R0402" value="330"/>
-<part name="LED1" library="led" deviceset="LED" device="CHIP-LED0805" value="Green LED"/>
+<part name="LED1" library="led" deviceset="LED" device="CHIPLED_0603" value="Green LED"/>
 <part name="R13" library="resistor" deviceset="R-US_" device="R0402" value="330"/>
 <part name="+3V9" library="supply1" deviceset="+3V3" device=""/>
