File: Hardware/v2/Board_R2_v2.brd (EAGLE design)
At the start: 100 x 80 mm, 67 parts, among them U1 EDISON_CONNECTOR_FULLMOUNTING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, U2 LAN9512-JZX, U3 MAX4995AAUT+, U4 EDISON_CONNECTOR_FULLHEADER, U5 USD-SOCKETNEW, U6 TXB0108

Commit message: Changed PoE module to accomodate USB_VBUS, changed Rectifiers, added level shifter
Parts:
- added C33, C34: 22uF, SparkFun-Capacitors:0805
- added C35: 47pF, SparkFun-Capacitors:0603-CAP
- added L3: 1.0uH, SparkFun-Passives:1210
- added R18: 120K, SparkFun-Resistors:0402-RES
- added U7: TPS62065, SparkFun-PowerIC:WSON-8-PAD
- B1, B2: value MB4S -> DF1510S; device rectifier:SOIC-4 -> PoEdev:DFS
- R16: value 0 -> 680K; device resistor:R1210 -> SparkFun-Resistors:0402-RES
- moved R16 109.2 mm to (-91.4, -44.5)
- moved B2 94.9 mm to (-81.3, -29.2)
- moved B1 86.4 mm to (-81.3, -17.8)
- renumbered AG9803MT to AG9805MT
Connections:
- new net N$32: C35.2, R16.1, R18.2, U7.4
- net GND: now also C33.2, C34.2, R18.1, U7.1, U7.3, U7.6, U7.PAD; no longer R16.2
- net N$14: now also L3.1, U7.2; no longer AG9805MT.P$4, R16.1
- net N$27: now also B1.~@1; no longer B1.~1
- net N$28: now also B1.~@2; no longer B1.~2
- net N$29: now also B2.~@1; no longer B2.~1
- net N$30: now also B2.~@2; no longer B2.~2
- net USB_VBUS: now also AG9805MT.P$1, AG9805MT.P$2, C30.1, C31.1, C32.1, C33.1, U7.5, U7.7, U7.8
- net VSYS: now also C34.1, C35.1, L3.2, R16.2; no longer AG9805MT.P$1, AG9805MT.P$2, C30.1, C31.1, C32.1
