File: Hardware/v2/PoE_Board.sch (EAGLE design)
At the start: 77 parts, among them U1 EDISON_CONNECTOR_FULLMOUNTING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, U2 LAN9512-JZX, U3 MAX4995AAUT+, U4 EDISON_CONNECTOR_FULLHEADER, U5 USD-SOCKETNEW, U6 TXB0108, U7 TPS62065

Commit message: PoE Board completed. Added Micro USB to schematic and board
Parts:
- added C37: 0.1uF, SparkFun-Capacitors:0.1UF-16V(+-10%)(0402)
- added C38, C39: 47pF, SparkFun-Capacitors:47PF-50V-5%(0603)
- added D3: RED, SparkFun-LED:LED-RED0603
- added D4: Yellow, SparkFun-LED:LED-YELLOW0603
- added JP1: (no value), SparkFun-Connectors:USB_MICROB_PLUGCONN-11752
- added R21: 0, SparkFun-Resistors:0OHM-1/10W-5%(0603)
- added R22, R23: 27, resistor:R-US_R0402
- added R24, R25: 100, resistor:R-US_R0402
- added R26, R27: (no value), resistor:R-US_R0402
- added U8: FT231XS-U, SparkFun-DigitalIC:FT231XS
- C36: value 22uF -> 0.1uF; device SparkFun-Capacitors:47PF-50V-5%(0603) -> SparkFun-Capacitors:0.1UF-16V(+-10%)(0402)
- R10: device resistor:R-US_R1210 -> SparkFun-Resistors:0OHM-1/10W-5%(0603)
- R20: value 25 -> 20; device resistor:R-US_R0402 -> resistor:R-US_R1206
Connections:
- removed net P22: U1.GP134_UART_2_RX, U4.GP134_UART_2_RX
- removed net P27: U1.GP135_UART_2_TX, U4.GP135_UART_2_TX
- new net +5V: C37.1, JP1.VCC, U8.VCC
- new net GP134_UART_2_RX: R24.2, U1.GP134_UART_2_RX, U4.GP134_UART_2_RX
- new net GP135_UART_2_TX: R25.2, U1.GP135_UART_2_TX, U4.GP135_UART_2_TX
- new net N$28: JP2.GND, R15.1, R21.2
- new net N$29: C38.1, JP1.D-, R22.1
- new net N$30: C39.1, JP1.D+, R23.1
- new net N$31: R22.2, U8.USBDM
- new net N$34: R23.2, U8.USBDP
- new net N$35: R24.1, U8.TXD
- new net N$36: R25.1, U8.RXD
- new net N$39: R27.1, U8.CBUS2
- new net N$40: R26.1, U8.CBUS1
- new net N$41: D3.C, R26.2
- new net N$42: D4.C, R27.2
- net 1.8V: now also C36.1, U8.!RESET, U8.VCCIO
- net CHASSGND: now also R10.2; no longer R10.1
- net GND: now also C37.2, C38.2, C39.2, JP1.GND, JP1.SHIELD, R10.1, R21.1, U8.GND@16, U8.GND@6; no longer JP2.GND, R10.2, R15.1
- net USB_VBUS: no longer C36.1
- net VSYS: now also D3.A, D4.A
Other:
- note added: "4"
- note added: "Added Micro USB and FDTI chip"
- note removed: "3.4"
- note removed: "Added downstream USB through hirose"
- moved on the sheet: C1, C10, C11, C12, C13, C14, C15, C16, C17, C2, C28, C29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

Commit message: Added ground fills. PoE: power planes around U7, diode for power through microB. Small: changed C26 to 2 caps, removed NP caps, removed test points, replaced crystal
Parts:
- added D5: MBRA140, SparkFun-DiscreteSemi:DIODE-SCHOTTKY-MBRA140
- U$1: device SparkFun-FreqCtrl:CRYSTAL-GROUNDED -> PoEdev:CRYSTAL-ESC-32
- renumbered RB1-125BHQ1A to X1
Connections:
- removed net USB_VBUS: AG9805MT.+VDC1, AG9805MT.+VDC2, C27.1, C30.1, C31.1, C32.1, C34.1, R20.2, U1.USB_VBUS, U3.IN, U4.USB_VBUS, U7.AVIN, U7.EN, U7.PVIN
- new net 5V: AG9805MT.+VDC1, AG9805MT.+VDC2, C30.1, C31.1, C32.1, C34.1, R20.2, U7.AVIN, U7.EN, U7.PVIN
- new net VBUS1: D5.A, JP1.VCC, U8.VCC
- net +5V: now also C27.1, D5.C, U1.USB_VBUS, U3.IN, U4.USB_VBUS; no longer JP1.VCC, U8.VCC
Other:
- note added: "Changed crystal, added diode for power over MicroB"
- note removed: "Added Micro USB and FDTI chip"

Commit message: Added LDO for power off VSYS, fixed SD card
Parts:
- removed R17: 10K, resistor:R-US_R0603
- removed TP1, TP2: TPTP20R, testpad:TPTP20R
- added C40, C41: 0.1uF, SparkFun-Capacitors:0.1UF-16V(+-10%)(0402)
- added C42, C43: 1.0uF, SparkFun-Capacitors:1.0UF-16V-10%(0402)
- added R28: 0, SparkFun-Resistors:0OHM-1/10W-5%(0603)
- added U9: (no value), PoEdev:MIC5353-XXYMT
- R26, R27: value (none) -> 1K
- U$1: device PoEdev:CRYSTAL-ESC-32 -> SparkFun-FreqCtrl:CRYSTAL-GROUNDED
Connections:
- removed net CLK24_OUT: TP1.TP, U2.CLK24_OUT
- removed net N$1: R17.1, U2.CLK24_EN
- new net ED3.3V: U1.3.3V@1, U1.3.3V@2, U4.3.3V@1, U4.3.3V@2
- new net N$32: JP1.SHIELD, R28.2
- new net N$38: C41.2, U9.BYP
- new net VCC: C40.1, C43.2, U9.EN, U9.VIN
- net +3V3: now also C42.1, U9.VOUT; no longer R17.2, U1.3.3V@1, U1.3.3V@2, U4.3.3V@1, U4.3.3V@2
- net GND: now also C40.2, C41.1, C42.2, C43.1, R28.1, U9.GND; no longer JP1.SHIELD, TP2.TP
Other:
- note added: "6"
- note added: "Added LDO for power off VSYS"
- note removed: "4"
- note removed: "Changed crystal, added diode for power over MicroB"
- moved on the sheet: AG9805MT, B1, B2, C28, C29, C30, C31, C32, C33, C34, C35, C36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

Commit message: Changed R20
Parts:
- R20: value 20 -> (none); device resistor:R-US_R1206 -> PoEdev:24OHM_1225
Other:
- note added: "6.1"
- note added: "Changed R20"
- note removed: "6"
- note removed: "Added LDO for power off VSYS"
Changed lines of the file:
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@@
 <part name="C39" library="SparkFun-Capacitors" deviceset="47PF-50V-5%(0603)" device="" value="47pF"/>
 <part name="SUPPLY6" library="SparkFun-Aesthetics" deviceset="1.8V" device=""/>
-<part name="R20" library="resistor" deviceset="R-US_" device="R1206" value="20"/>
 <part name="VSYS" library="supply1" deviceset="VCC" device="" value="VSYS"/>
 <part name="VSYS1" library="supply1" deviceset="VCC" device="" value="VSYS"/>
@@
 <part name="GND41" library="supply1" deviceset="GND" device=""/>
 <part name="GND42" library="supply1" deviceset="GND" device=""/>
+<part name="R20" library="PoEdev" deviceset="24OHM_1225" device=""/>
 </parts>
 <sheets>
@@
 <text x="292.1" y="96.52" size="1.778" layer="91">All Resistor Tolerances are 1% unless otherwise specified</text>
 <text x="327.66" y="27.94" size="3.048" layer="91">Ethernet/USB Block for Intel Edison</text>
-<text x="414.02" y="7.62" size="3.81" layer="91">6</text>
-<text x="327.66" y="7.62" size="1.778" layer="91">Added LDO for power off VSYS</text>
+<text x="414.02" y="7.62" size="3.81" layer="91">6.1</text>
+<text x="327.66" y="7.62" size="1.778" layer="91">Changed R20</text>
 <text x="327.406" y="11.176" size="2.54" layer="91">-----------------------REVISION NOTES</text>
 <text x="307.34" y="165.1" size="1.27" layer="91">Add 15pF capacitors in
@@
 </instance>
 <instance part="SUPPLY6" gate="G$1" x="12.7" y="76.2"/>
-<instance part="R20" gate="G$1" x="340.36" y="55.88" smashed="yes" rot="R90">
-<attribute name="NAME" x="342.6714" y="49.276" size="1.778" layer="95" rot="R90"/>
-<attribute name="VALUE" x="343.408" y="57.912" size="1.778" layer="96" rot="R90"/>
-</instance>
 <instance part="VSYS" gate="VCC" x="261.62" y="68.58" smashed="yes">
 <attribute name="VALUE" x="264.16" y="71.12" size="1.778" layer="96" rot="R180"/>
@@
 <instance part="GND41" gate="1" x="170.18" y="63.5"/>
 <instance part="GND42" gate="1" x="177.8" y="63.5"/>
+<instance part="R20" gate="G$1" x="340.36" y="55.88" rot="R90"/>
 </instances>
 <busses>
@@
 </segment>
 <segment>
-<pinref part="R20" gate="G$1" pin="1"/>
 <pinref part="GND24" gate="1" pin="GND"/>
 <wire x1="340.36" y1="43.18" x2="340.36" y2="48.26" width="0.1524" layer="91"/>
@@
 <junction x="347.98" y="48.26"/>
 <junction x="340.36" y="48.26"/>
+<pinref part="R20" gate="G$1" pin="1"/>
 </segment>
 <segment>
@@
 <junction x="337.82" y="60.96"/>
 <pinref part="C34" gate="G$1" pin="1"/>
-<junction x="340.36" y="60.96"/>
 <pinref part="5V" gate="1" pin="+5V"/>
 <pinref part="R20" gate="G$1" pin="2"/>
-</segment>
-</net>
+<junction x="340.36" y="60.96"/>
+</segment>
+</net>
